File: lamp copy.brd (EAGLE design)
At the start: 127.3 x 38.1 mm, 53 parts

Commit message: Fiddled the board xml by hand to place the last few parts. Some more adjustment of traces. Added a low-noise cap to the 5v regulator.
Parts:
- added C3: 10nF, Barebones-Arduino:0805
- C1: value (none) -> 1µF
- C2: value (none) -> 2.2µF
- moved U$2 53.4 mm to (120.7, 5.08)
- moved U$3 53.4 mm to (120.7, 19.1)
- moved U$4 53.4 mm to (120.7, 33.0)
- moved R1 53.4 mm to (116.2, 33.0)
- moved U$5 39.6 mm to (108.0, 5.08)
- moved U$6 39.6 mm to (108.0, 19.1)
- moved U$7 39.6 mm to (108.0, 33.0)
- moved R2 39.6 mm to (103.5, 33.0)
- moved C2 1.62 mm to (67.3, 4.13), turned to 180 degrees
- moved C1 1.27 mm to (58.7, 5.71)
- moved LR 1.27 mm to (62.2, 5.71)
Connections:
- new net N$46: C3.1, LR.P$4
- net GND: now also C3.2
Routing:
- net N$50: track 12.5 -> 0.00 mm
- net N$53: track 12.5 -> 0.00 mm
- net N$49: track 12.5 -> 0.00 mm
- net N$54: track 12.2 -> 0.00 mm
- net N$6: track 0.00 -> 11.6 mm
- net N$3: track 0.00 -> 11.6 mm
- net N$4: track 0.00 -> 11.6 mm
- net N$1: track 0.00 -> 11.6 mm
- net N$15: track 14.1 -> 22.4 mm
- net N$51: track 5.29 -> 0.00 mm, vias 1 -> 0
- net N$45: track 5.29 -> 0.00 mm, vias 1 -> 0
- net N$2: track 0.00 -> 4.65 mm, vias 0 -> 1
- net N$5: track 0.00 -> 4.65 mm, vias 0 -> 1
- net N$46: track 0.00 -> 2.99 mm
- net +12V: track 179.0 -> 178.0 mm
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Other:
- board size 127.3 x 38.1 mm -> 127 x 38.1 mm
- board text added: "C1"
- board text added: "C2"
- board text added: "C3"
- board text added: "LR"
- board text added: "R1"
- board text added: "R10"
- board text added: "R2"
- board text added: "R3"
- board text added: "R4"
- board text added: "R5"
- board text added: "R6"
- board text added: "R7"
- board text added: "R8"
- board text added: "R9"
