File: lamp.brd (EAGLE design)
At the start: 127 x 38.1 mm, 57 parts

Commit message: fixed led vsupply to be from the pfet added in last commit instead of straight from +12v
Connections:
- net +12V: no longer TA.P$10, U$1.P$2, U$11.P$2, U$16.P$2, U$2.P$2, U$20.P$2, U$23.P$2, U$26.P$2, U$29.P$2, U$5.P$2, U$8.P$2
- net N$45: now also TA.P$10, U$1.P$2, U$11.P$2, U$16.P$2, U$2.P$2, U$20.P$2, U$23.P$2, U$26.P$2, U$29.P$2, U$5.P$2, U$8.P$2
Routing:
- net N$45: track 0.00 -> 178.4 mm, vias 0 -> 2
- net +12V: track 178.4 -> 0.00 mm, vias 2 -> 0
Changed lines of the file:
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@@
 </signal>
 <signal name="+12V">
-<contactref element="U$2" pad="P$2"/>
-<contactref element="U$5" pad="P$2"/>
-<contactref element="U$8" pad="P$2"/>
-<contactref element="U$11" pad="P$2"/>
-<contactref element="U$20" pad="P$2"/>
-<contactref element="U$23" pad="P$2"/>
-<contactref element="U$26" pad="P$2"/>
-<contactref element="U$29" pad="P$2"/>
-<wire x1="7.3025" y1="3.4925" x2="7.3025" y2="1.27" width="1.27" layer="1"/>
-<wire x1="7.3025" y1="1.27" x2="20.0025" y2="1.27" width="1.27" layer="1"/>
-<wire x1="20.0025" y1="1.27" x2="32.7025" y2="1.27" width="1.27" layer="1"/>
-<wire x1="32.7025" y1="1.27" x2="63.5" y2="1.27" width="1.27" layer="1"/>
-<wire x1="58.1025" y1="1.27" x2="58.1025" y2="3.4925" width="1.27" layer="1"/>
-<wire x1="20.0025" y1="3.4925" x2="20.0025" y2="1.27" width="1.27" layer="1"/>
-<wire x1="32.7025" y1="3.4925" x2="32.7025" y2="1.27" width="1.27" layer="1"/>
-<wire x1="45.4025" y1="3.4925" x2="45.4025" y2="1.27" width="1.27" layer="1"/>
-<wire x1="58.1025" y1="1.27" x2="63.5" y2="1.27" width="1.27" layer="1"/>
-<wire x1="63.5" y1="1.27" x2="70.8025" y2="1.27" width="1.27" layer="1"/>
-<wire x1="70.8025" y1="1.27" x2="83.5025" y2="1.27" width="1.27" layer="1"/>
-<wire x1="83.5025" y1="1.27" x2="121.6025" y2="1.27" width="1.27" layer="1"/>
-<wire x1="70.8025" y1="3.4925" x2="70.8025" y2="1.27" width="1.27" layer="1"/>
-<wire x1="83.5025" y1="3.4925" x2="83.5025" y2="1.27" width="1.27" layer="1"/>
-<wire x1="63.5" y1="22.86" x2="63.5" y2="1.27" width="0.6096" layer="1"/>
-<via x="63.5" y="22.86" extent="1-16" drill="0.5"/>
-<contactref element="TA" pad="P$10"/>
-<wire x1="58.42" y1="25.655" x2="58.42" y2="24.13" width="0.6096" layer="16"/>
-<wire x1="58.42" y1="24.13" x2="59.69" y2="22.86" width="0.6096" layer="16"/>
-<wire x1="59.69" y1="22.86" x2="63.5" y2="22.86" width="0.6096" layer="16"/>
-<contactref element="U$1" pad="P$2"/>
-<contactref element="U$16" pad="P$2"/>
-<via x="63.5" y="1.27" extent="1-16" drill="0.5"/>
-<wire x1="62.23" y1="4.7625" x2="62.23" y2="6.0325" width="0.4064" layer="16"/>
-<wire x1="62.23" y1="6.0325" x2="61.595" y2="6.6675" width="0.4064" layer="16"/>
-<wire x1="61.595" y1="6.6675" x2="60.96" y2="6.6675" width="0.4064" layer="16"/>
-<wire x1="63.5" y1="1.27" x2="62.23" y2="2.54" width="0.4064" layer="16"/>
-<wire x1="62.23" y1="2.54" x2="62.23" y2="4.7625" width="0.4064" layer="16"/>
-<wire x1="62.23" y1="4.7625" x2="58.7375" y2="4.7625" width="0.4064" layer="16"/>
-<wire x1="121.6025" y1="1.27" x2="121.6025" y2="3.4925" width="1.27" layer="1"/>
-<wire x1="108.9025" y1="3.4925" x2="108.9025" y2="1.5875" width="1.27" layer="1"/>
 <contactref element="U$19" pad="P$3"/>
 <contactref element="U$32" pad="P$1"/>
-<wire x1="96.2025" y1="3.4925" x2="108.9025" y2="3.4925" width="0" layer="19" extent="1-1"/>
-<wire x1="121.6025" y1="3.4925" x2="108.9025" y2="3.4925" width="0" layer="19" extent="1-1"/>
-<wire x1="-2.54" y1="3.86" x2="7.3025" y2="3.4925" width="0" layer="19" extent="1-1"/>
-<wire x1="-7.62" y1="1.27" x2="-2.54" y2="3.86" width="0" layer="19" extent="1-1"/>
-<wire x1="45.4025" y1="3.4925" x2="58.1025" y2="3.4925" width="0" layer="19" extent="1-1"/>
+<wire x1="-2.54" y1="3.86" x2="-7.62" y2="1.27" width="0" layer="19" extent="1-1"/>
 </signal>
 <signal name="N$33">
@@
 <contactref element="VR" pad="P$1"/>
 <contactref element="U$19" pad="P$2"/>
-<wire x1="60.91" y1="4.795" x2="60.91" y2="6.635" width="0" layer="19" extent="16-16"/>
-<wire x1="58.7375" y1="4.865" x2="60.91" y2="4.795" width="0" layer="19" extent="16-16"/>
-<wire x1="-1.62" y1="1.17" x2="58.7375" y2="4.865" width="0" layer="19" extent="1-16"/>
+<contactref element="U$2" pad="P$2"/>
+<contactref element="U$5" pad="P$2"/>
+<contactref element="U$8" pad="P$2"/>
+<contactref element="U$11" pad="P$2"/>
+<contactref element="U$20" pad="P$2"/>
+<contactref element="U$23" pad="P$2"/>
+<contactref element="U$26" pad="P$2"/>
+<contactref element="U$29" pad="P$2"/>
+<contactref element="TA" pad="P$10"/>
+<contactref element="U$1" pad="P$2"/>
+<contactref element="U$16" pad="P$2"/>
+<wire x1="7.3025" y1="3.4925" x2="7.3025" y2="1.27" width="1.27" layer="1"/>
+<wire x1="7.3025" y1="1.27" x2="20.0025" y2="1.27" width="1.27" layer="1"/>
+<wire x1="20.0025" y1="1.27" x2="32.7025" y2="1.27" width="1.27" layer="1"/>
+<wire x1="32.7025" y1="1.27" x2="63.5" y2="1.27" width="1.27" layer="1"/>
+<wire x1="58.1025" y1="1.27" x2="58.1025" y2="3.4925" width="1.27" layer="1"/>
+<wire x1="20.0025" y1="3.4925" x2="20.0025" y2="1.27" width="1.27" layer="1"/>
+<wire x1="32.7025" y1="3.4925" x2="32.7025" y2="1.27" width="1.27" layer="1"/>
+<wire x1="45.4025" y1="3.4925" x2="45.4025" y2="1.27" width="1.27" layer="1"/>
+<wire x1="58.1025" y1="1.27" x2="63.5" y2="1.27" width="1.27" layer="1"/>
+<wire x1="63.5" y1="1.27" x2="70.8025" y2="1.27" width="1.27" layer="1"/>
+<wire x1="70.8025" y1="1.27" x2="83.5025" y2="1.27" width="1.27" layer="1"/>
+<wire x1="83.5025" y1="1.27" x2="121.6025" y2="1.27" width="1.27" layer="1"/>
+<wire x1="70.8025" y1="3.4925" x2="70.8025" y2="1.27" width="1.27" layer="1"/>
+<wire x1="83.5025" y1="3.4925" x2="83.5025" y2="1.27" width="1.27" layer="1"/>
+<wire x1="63.5" y1="22.86" x2="63.5" y2="1.27" width="0.6096" layer="1"/>
+<via x="63.5" y="22.86" extent="1-16" drill="0.5"/>
+<wire x1="58.42" y1="25.655" x2="58.42" y2="24.13" width="0.6096" layer="16"/>
+<wire x1="58.42" y1="24.13" x2="59.69" y2="22.86" width="0.6096" layer="16"/>
+<wire x1="59.69" y1="22.86" x2="63.5" y2="22.86" width="0.6096" layer="16"/>
+<via x="63.5" y="1.27" extent="1-16" drill="0.5"/>
+<wire x1="62.23" y1="4.7625" x2="62.23" y2="6.0325" width="0.4064" layer="16"/>
+<wire x1="62.23" y1="6.0325" x2="61.595" y2="6.6675" width="0.4064" layer="16"/>
+<wire x1="61.595" y1="6.6675" x2="60.96" y2="6.6675" width="0.4064" layer="16"/>
+<wire x1="63.5" y1="1.27" x2="62.23" y2="2.54" width="0.4064" layer="16"/>
+<wire x1="62.23" y1="2.54" x2="62.23" y2="4.7625" width="0.4064" layer="16"/>
+<wire x1="62.23" y1="4.7625" x2="58.7375" y2="4.7625" width="0.4064" layer="16"/>
+<wire x1="121.6025" y1="1.27" x2="121.6025" y2="3.4925" width="1.27" layer="1"/>
+<wire x1="108.9025" y1="3.4925" x2="108.9025" y2="1.5875" width="1.27" layer="1"/>
+<wire x1="96.2025" y1="3.4925" x2="108.9025" y2="3.4925" width="0" layer="19" extent="1-1"/>
+<wire x1="121.6025" y1="3.4925" x2="108.9025" y2="3.4925" width="0" layer="19" extent="1-1"/>
+<wire x1="60.91" y1="6.635" x2="60.96" y2="6.6675" width="0" layer="19" extent="16-16"/>
+<wire x1="58.7375" y1="4.865" x2="58.7375" y2="4.7625" width="0" layer="19" extent="16-16"/>
+<wire x1="60.91" y1="4.795" x2="62.23" y2="4.7625" width="0" layer="19" extent="16-16"/>
+<wire x1="-1.62" y1="1.17" x2="7.3025" y2="1.27" width="0" layer="19" extent="1-1"/>
+<wire x1="45.4025" y1="3.4925" x2="58.1025" y2="3.4925" width="0" layer="19" extent="1-1"/>
 </signal>
 </signals>
